File: hardware/TireTempSensor_v2.0/IRSensor.kicad_sch (KiCad schematic)
At the start: 0 parts

Commit message: PFET & buck caps models
Parts:
- added C?: 100n, Capacitor_SMD:C_0603_1608Metric, symbol Device:C
- added FB?: 60R@100MHz, Inductor_SMD:L_0603_1608Metric, symbol Device:FerriteBead_Small
- added IC?: MLX90621ESF-BAB-000-SP, MLX:MLX90621ESFBAB000SP, symbol MLX90621ESF-BAB-000-SP:MLX90621ESF-BAB-000-SP
- added R? (x2): 4k7, Resistor_SMD:R_0603_1608Metric, symbol Device:R_US
Connections:
- new net: C?.1, FB?.2, IC?.3 (VDD)
- new net +2V6: FB?.1
- new net +3V3: R?.1, R?.1
- new net GND: C?.2, IC?.4 (GND)
- new net SCL: IC?.1 (SCL), R?.2
- new net SDA: IC?.2 (SDA), R?.2
Other:
- title: (none) -> IR Sensor
Changed lines of the file:
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@@
 (kicad_sch (version 20211123) (generator eeschema)
   (paper "A4")
+  (title_block
+    (title "IR Sensor")
+  )
+  (junction (at 125.73 100.33) (diameter 0) (color 0 0 0 0)
+  )
+  (junction (at 130.81 115.57) (diameter 0) (color 0 0 0 0)
+  )
+  (junction (at 151.13 100.33) (diameter 0) (color 0 0 0 0)
+  )
+  (junction (at 138.43 85.09) (diameter 0) (color 0 0 0 0)
+  )
+  (junction (at 144.78 72.39) (diameter 0) (color 0 0 0 0)
+  )
+  (wire (pts (xy 138.43 76.2) (xy 138.43 72.39))
+    (stroke (width 0) (type default) (color 0 0 0 0))
+  )
+  (wire (pts (xy 138.43 83.82) (xy 138.43 85.09))
+    (stroke (width 0) (type default) (color 0 0 0 0))
+  )
+  (wire (pts (xy 144.78 72.39) (xy 151.13 72.39))
+    (stroke (width 0) (type default) (color 0 0 0 0))
+  )
+  (wire (pts (xy 125.73 115.57) (xy 130.81 115.57))
+    (stroke (width 0) (type default) (color 0 0 0 0))
+  )
+  (wire (pts (xy 151.13 72.39) (xy 151.13 76.2))
+    (stroke (width 0) (type default) (color 0 0 0 0))
+  )
+  (wire (pts (xy 151.13 100.33) (xy 160.02 100.33))
+    (stroke (width 0) (type default) (color 0 0 0 0))
+  )
+  (wire (pts (xy 125.73 110.49) (xy 125.73 115.57))
+    (stroke (width 0) (type default) (color 0 0 0 0))
+  )
+  (wire (pts (xy 125.73 91.44) (xy 125.73 92.71))
+    (stroke (width 0) (type default) (color 0 0 0 0))
+  )
+  (wire (pts (xy 144.78 69.85) (xy 144.78 72.39))
+    (stroke (width 0) (type default) (color 0 0 0 0))
+  )
+  (wire (pts (xy 130.81 115.57) (xy 130.81 118.11))
+    (stroke (width 0) (type default) (color 0 0 0 0))
+  )
+  (wire (pts (xy 125.73 97.79) (xy 125.73 100.33))
+    (stroke (width 0) (type default) (color 0 0 0 0))
+  )
+  (wire (pts (xy 125.73 102.87) (xy 125.73 100.33))
+    (stroke (width 0) (type default) (color 0 0 0 0))
+  )
+  (wire (pts (xy 138.43 85.09) (xy 160.02 85.09))
+    (stroke (width 0) (type default) (color 0 0 0 0))
+  )
+  (wire (pts (xy 130.81 115.57) (xy 138.43 115.57))
+    (stroke (width 0) (type default) (color 0 0 0 0))
+  )
+  (wire (pts (xy 151.13 83.82) (xy 151.13 100.33))
+    (stroke (width 0) (type default) (color 0 0 0 0))
+  )
+  (wire (pts (xy 138.43 72.39) (xy 144.78 72.39))
+    (stroke (width 0) (type default) (color 0 0 0 0))
+  )
+  (hierarchical_label "SCL" (shape input) (at 160.02 100.33 0)
+    (effects (font (size 1.27 1.27)) (justify left))
+  )
+  (hierarchical_label "SDA" (shape bidirectional) (at 160.02 85.09 0)
+    (effects (font (size 1.27 1.27)) (justify left))
+  )
+  (symbol (lib_id "Device:R_US") (at 151.13 80.01 0) (unit 1)
+    (in_bom yes) (on_board yes) (fields_autoplaced)
+    (property "Reference" "R?" (id 0) (at 153.67 78.7399 0)
+      (effects (font (size 1.27 1.27)) (justify left))
+    )
+    (property "Value" "4k7" (id 1) (at 153.67 81.2799 0)
+      (effects (font (size 1.27 1.27)) (justify left))
+    )
+    (property "Footprint" "Resistor_SMD:R_0603_1608Metric" (id 2) (at 152.146 80.264 90)
+      (effects (font (size 1.27 1.27)) hide)
+    )
+    (property "Datasheet" "~" (id 3) (at 151.13 80.01 0)
+      (effects (font (size 1.27 1.27)) hide)
+    )
+    (pin "1")
+    (pin "2")
+  )
+  (symbol (lib_id "power:+3V3") (at 144.78 69.85 0) (unit 1)
+    (in_bom yes) (on_board yes) (fields_autoplaced)
+    (property "Reference" "#PWR?" (id 0) (at 144.78 73.66 0)
+      (effects (font (size 1.27 1.27)) hide)
+    )
+    (property "Value" "+3V3" (id 1) (at 144.78 64.77 0))
+    (property "Footprint" "" (id 2) (at 144.78 69.85 0)
+      (effects (font (size 1.27 1.27)) hide)
+    )
+    (property "Datasheet" "" (id 3) (at 144.78 69.85 0)
+      (effects (font (size 1.27 1.27)) hide)
+    )
+    (pin "1")
+  )
+  (symbol (lib_id "Device:R_US") (at 138.43 80.01 0) (unit 1)
+    (in_bom yes) (on_board yes) (fields_autoplaced)
+    (property "Reference" "R?" (id 0) (at 140.97 78.7399 0)
+      (effects (font (size 1.27 1.27)) (justify left))
+    )
+    (property "Value" "4k7" (id 1) (at 140.97 81.2799 0)
+      (effects (font (size 1.27 1.27)) (justify left))
+    )
+    (property "Footprint" "Resistor_SMD:R_0603_1608Metric" (id 2) (at 139.446 80.264 90)
+      (effects (font (size 1.27 1.27)) hide)
+    )
+    (property "Datasheet" "~" (id 3) (at 138.43 80.01 0)
+      (effects (font (size 1.27 1.27)) hide)
+    )
+    (pin "1")
+    (pin "2")
+  )
+  (symbol (lib_id "power:GND") (at 130.81 118.11 0) (unit 1)
+    (in_bom yes) (on_board yes) (fields_autoplaced)
+    (property "Reference" "#PWR?" (id 0) (at 130.81 124.46 0)
+      (effects (font (size 1.27 1.27)) hide)
+    )
+    (property "Value" "GND" (id 1) (at 130.81 123.19 0))
+    (property "Footprint" "" (id 2) (at 130.81 118.11 0)
+      (effects (font (size 1.27 1.27)) hide)
+    )
+    (property "Datasheet" "" (id 3) (at 130.81 118.11 0)
+      (effects (font (size 1.27 1.27)) hide)
+    )
+    (pin "1")
+  )
+  (symbol (lib_id "power:+2V6") (at 125.73 91.44 0) (unit 1)
+    (in_bom yes) (on_board yes) (fields_autoplaced)
+    (property "Reference" "#PWR?" (id 0) (at 125.73 95.25 0)
+      (effects (font (size 1.27 1.27)) hide)
+    )
+    (property "Value" "+2V6" (id 1) (at 125.73 86.36 0))
+    (property "Footprint" "" (id 2) (at 125.73 91.44 0)
+      (effects (font (size 1.27 1.27)) hide)
+    )
+    (property "Datasheet" "" (id 3) (at 125.73 91.44 0)
+      (effects (font (size 1.27 1.27)) hide)
+    )
+    (pin "1")
+  )
+  (symbol (lib_id "MLX90621ESF-BAB-000-SP:MLX90621ESF-BAB-000-SP") (at 125.73 100.33 0) (unit 1)
+    (in_bom yes) (on_board yes)
+    (property "Reference" "IC?" (id 0) (at 149.86 110.49 0))
+    (property "Value" "MLX90621ESF-BAB-000-SP" (id 1) (at 154.94 114.3 0))
+    (property "Footprint" "MLX:MLX90621ESFBAB000SP" (id 2) (at 147.32 90.17 0)
+      (effects (font (size 1.27 1.27)) (justify left) hide)
+    )
+    (property "Datasheet" "https://www.melexis.com/-/media/files/documents/datasheets/mlx90621-datasheet-melexis.pdf" (id 3) (at 147.32 92.71 0)
+      (effects (font (size 1.27 1.27)) (justify left) hide)
+    )
+    (property "Description" "Board Mount Temperature Sensors 16X4 thermal array sensor, 3Volt, 60deg total FOV" (id 4) (at 147.32 95.25 0)
+      (effects (font (size 1.27 1.27)) (justify left) hide)
+    )
+    (property "Height" "11.4" (id 5) (at 147.32 97.79 0)
+      (effects (font (size 1.27 1.27)) (justify left) hide)
+    )
+    (property "Manufacturer_Name" "Melexis" (id 6) (at 147.32 100.33 0)
+      (effects (font (size 1.27 1.27)) (justify left) hide)
+    )
+    (property "Manufacturer_Part_Number" "MLX90621ESF-BAB-000-SP" (id 7) (at 147.32 102.87 0)
+      (effects (font (size 1.27 1.27)) (justify left) hide)
+    )
+    (property "Mouser Part Number" "482-90621ESFBAB000SP" (id 8) (at 147.32 105.41 0)
+      (effects (font (size 1.27 1.27)) (justify left) hide)
+    )
+    (property "Mouser Price/Stock" "https://www.mouser.co.uk/ProductDetail/Melexis/MLX90621ESF-BAB-000-SP/?qs=KuGPmAKtFKVFHvV1D3wVtw%3D%3D" (id 9) (at 147.32 107.95 0)
+      (effects (font (size 1.27 1.27)) (justify left) hide)
+    )
+    (property "Arrow Part Number" "" (id 10) (at 147.32 110.49 0)
+      (effects (font (size 1.27 1.27)) (justify left) hide)
+    )
+    (property "Arrow Price/Stock" "" (id 11) (at 147.32 113.03 0)
+      (effects (font (size 1.27 1.27)) (justify left) hide)
+    )
+    (pin "1")
+    (pin "2")
+    (pin "3")
+    (pin "4")
+  )
+  (symbol (lib_id "Device:FerriteBead_Small") (at 125.73 95.25 0) (unit 1)
+    (in_bom yes) (on_board yes)
+    (property "Reference" "FB?" (id 0) (at 118.11 93.98 0)
+      (effects (font (size 1.27 1.27)) (justify left))
+    )
+    (property "Value" "60R@100MHz" (id 1) (at 109.22 96.52 0)
+      (effects (font (size 1.27 1.27)) (justify left))
+    )
+    (property "Footprint" "Inductor_SMD:L_0603_1608Metric" (id 2) (at 123.952 95.25 90)
+      (effects (font (size 1.27 1.27)) hide)
+    )
+    (property "Datasheet" "~" (id 3) (at 125.73 95.25 0)
+      (effects (font (size 1.27 1.27)) hide)
+    )
+    (pin "1")
+    (pin "2")
+  )
+  (symbol (lib_id "Device:C") (at 125.73 106.68 0) (unit 1)
+    (in_bom yes) (on_board yes)
+    (property "Reference" "C?" (id 0) (at 118.11 105.41 0)
+      (effects (font (size 1.27 1.27)) (justify left))
+    )
+    (property "Value" "100n" (id 1) (at 116.84 107.95 0)
+      (effects (font (size 1.27 1.27)) (justify left))
+    )
+    (property "Footprint" "Capacitor_SMD:C_0603_1608Metric" (id 2) (at 126.6952 110.49 0)
+      (effects (font (size 1.27 1.27)) hide)
+    )
+    (property "Datasheet" "~" (id 3) (at 125.73 106.68 0)
+      (effects (font (size 1.27 1.27)) hide)
+    )
+    (pin "1")
+    (pin "2")
+  )
 )

Commit message: erc tests passed
Parts:
- removed IC?: MLX90621ESF-BAB-000-SP, MLX:MLX90621ESFBAB000SP, symbol MLX90621ESF-BAB-000-SP:MLX90621ESF-BAB-000-SP
- added IC2: MLX90621ESF-BAB-000-SP, MLX90621ESFBAB000SP, symbol irsensor:MLX90621ESF-BAB-000-SP
- gave numbers to parts that had none: 4
Connections:
- net GND: now also IC2.4 (GND)
- net SCL: now also IC2.1 (SCL)
- net SDA: now also IC2.2 (SDA)
- net at C17.1, FB3.2: now also IC2.3 (VDD)
Changed lines of the file:
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@@
     (title "IR Sensor")
   )
+  (junction (at 130.81 115.57) (diameter 0) (color 0 0 0 0)
+  )
+  (junction (at 151.13 100.33) (diameter 0) (color 0 0 0 0)
+  )
   (junction (at 125.73 100.33) (diameter 0) (color 0 0 0 0)
   )
-  (junction (at 130.81 115.57) (diameter 0) (color 0 0 0 0)
-  )
-  (junction (at 151.13 100.33) (diameter 0) (color 0 0 0 0)
-  )
   (junction (at 138.43 85.09) (diameter 0) (color 0 0 0 0)
   )
@@
     (stroke (width 0) (type default) (color 0 0 0 0))
   )
+  (wire (pts (xy 125.73 100.33) (xy 125.73 102.87))
+    (stroke (width 0) (type default) (color 0 0 0 0))
+  )
   (wire (pts (xy 151.13 100.33) (xy 160.02 100.33))
     (stroke (width 0) (type default) (color 0 0 0 0))
@@
   )
   (wire (pts (xy 125.73 97.79) (xy 125.73 100.33))
-    (stroke (width 0) (type default) (color 0 0 0 0))
-  )
-  (wire (pts (xy 125.73 102.87) (xy 125.73 100.33))
     (stroke (width 0) (type default) (color 0 0 0 0))
   )
@@
   (symbol (lib_id "Device:R_US") (at 151.13 80.01 0) (unit 1)
     (in_bom yes) (on_board yes) (fields_autoplaced)
-    (property "Reference" "R?" (id 0) (at 153.67 78.7399 0)
+    (property "Reference" "R6" (id 0) (at 153.67 78.7399 0)
       (effects (font (size 1.27 1.27)) (justify left))
     )
@@
   (symbol (lib_id "power:+3V3") (at 144.78 69.85 0) (unit 1)
     (in_bom yes) (on_board yes) (fields_autoplaced)
-    (property "Reference" "#PWR?" (id 0) (at 144.78 73.66 0)
+    (property "Reference" "#PWR0128" (id 0) (at 144.78 73.66 0)
       (effects (font (size 1.27 1.27)) hide)
     )
@@
   (symbol (lib_id "Device:R_US") (at 138.43 80.01 0) (unit 1)
     (in_bom yes) (on_board yes) (fields_autoplaced)
-    (property "Reference" "R?" (id 0) (at 140.97 78.7399 0)
+    (property "Reference" "R5" (id 0) (at 140.97 78.7399 0)
       (effects (font (size 1.27 1.27)) (justify left))
     )
@@
   (symbol (lib_id "power:GND") (at 130.81 118.11 0) (unit 1)
     (in_bom yes) (on_board yes) (fields_autoplaced)
-    (property "Reference" "#PWR?" (id 0) (at 130.81 124.46 0)
+    (property "Reference" "#PWR0126" (id 0) (at 130.81 124.46 0)
       (effects (font (size 1.27 1.27)) hide)
     )
@@
     (pin "1")
   )
-  (symbol (lib_id "power:+2V6") (at 125.73 91.44 0) (unit 1)
-    (in_bom yes) (on_board yes) (fields_autoplaced)
-    (property "Reference" "#PWR?" (id 0) (at 125.73 95.25 0)
+  (symbol (lib_id "Device:FerriteBead_Small") (at 125.73 95.25 0) (unit 1)
+    (in_bom yes) (on_board yes)
+    (property "Reference" "FB3" (id 0) (at 118.11 93.98 0)
+      (effects (font (size 1.27 1.27)) (justify left))
+    )
+    (property "Value" "60R@100MHz" (id 1) (at 109.22 96.52 0)
+      (effects (font (size 1.27 1.27)) (justify left))
+    )
+    (property "Footprint" "Inductor_SMD:L_0603_1608Metric" (id 2) (at 123.952 95.25 90)
+      (effects (font (size 1.27 1.27)) hide)
+    )
+    (property "Datasheet" "~" (id 3) (at 125.73 95.25 0)
+      (effects (font (size 1.27 1.27)) hide)
+    )
+    (pin "1")
+    (pin "2")
+  )
+  (symbol (lib_id "Device:C") (at 125.73 106.68 0) (unit 1)
+    (in_bom yes) (on_board yes)
+    (property "Reference" "C17" (id 0) (at 118.11 105.41 0)
+      (effects (font (size 1.27 1.27)) (justify left))
+    )
+    (property "Value" "100n" (id 1) (at 116.84 107.95 0)
+      (effects (font (size 1.27 1.27)) (justify left))
+    )
+    (property "Footprint" "Capacitor_SMD:C_0603_1608Metric" (id 2) (at 126.6952 110.49 0)
+      (effects (font (size 1.27 1.27)) hide)
+    )
+    (property "Datasheet" "~" (id 3) (at 125.73 106.68 0)
+      (effects (font (size 1.27 1.27)) hide)
+    )
+    (pin "1")
+    (pin "2")
+  )
+  (symbol (lib_id "2v6:+2V6") (at 125.73 91.44 0) (unit 1)
+    (in_bom yes) (on_board yes) (fields_autoplaced)
+    (property "Reference" "#PWR0127" (id 0) (at 125.73 95.25 0)
       (effects (font (size 1.27 1.27)) hide)
     )
@@
     (pin "1")
   )
-  (symbol (lib_id "MLX90621ESF-BAB-000-SP:MLX90621ESF-BAB-000-SP") (at 125.73 100.33 0) (unit 1)
+  (symbol (lib_id "irsensor:MLX90621ESF-BAB-000-SP") (at 125.73 100.33 0) (unit 1)
     (in_bom yes) (on_board yes)
-    (property "Reference" "IC?" (id 0) (at 149.86 110.49 0))
-    (property "Value" "MLX90621ESF-BAB-000-SP" (id 1) (at 154.94 114.3 0))
-    (property "Footprint" "MLX:MLX90621ESFBAB000SP" (id 2) (at 147.32 90.17 0)
+    (property "Reference" "IC2" (id 0) (at 156.21 110.49 0))
+    (property "Value" "MLX90621ESF-BAB-000-SP" (id 1) (at 156.21 113.03 0))
+    (property "Footprint" "MLX90621ESFBAB000SP" (id 2) (at 147.32 90.17 0)
       (effects (font (size 1.27 1.27)) (justify left) hide)
     )
@@
     (pin "4")
   )
-  (symbol (lib_id "Device:FerriteBead_Small") (at 125.73 95.25 0) (unit 1)
-    (in_bom yes) (on_board yes)
-    (property "Reference" "FB?" (id 0) (at 118.11 93.98 0)
-      (effects (font (size 1.27 1.27)) (justify left))
-    )
-    (property "Value" "60R@100MHz" (id 1) (at 109.22 96.52 0)
-      (effects (font (size 1.27 1.27)) (justify left))
-    )
-    (property "Footprint" "Inductor_SMD:L_0603_1608Metric" (id 2) (at 123.952 95.25 90)
-      (effects (font (size 1.27 1.27)) hide)
-    )
-    (property "Datasheet" "~" (id 3) (at 125.73 95.25 0)
-      (effects (font (size 1.27 1.27)) hide)
-    )
-    (pin "1")
-    (pin "2")
-  )
-  (symbol (lib_id "Device:C") (at 125.73 106.68 0) (unit 1)
-    (in_bom yes) (on_board yes)
-    (property "Reference" "C?" (id 0) (at 118.11 105.41 0)
-      (effects (font (size 1.27 1.27)) (justify left))
-    )
-    (property "Value" "100n" (id 1) (at 116.84 107.95 0)
-      (effects (font (size 1.27 1.27)) (justify left))
-    )
-    (property "Footprint" "Capacitor_SMD:C_0603_1608Metric" (id 2) (at 126.6952 110.49 0)
-      (effects (font (size 1.27 1.27)) hide)
-    )
-    (property "Datasheet" "~" (id 3) (at 125.73 106.68 0)
-      (effects (font (size 1.27 1.27)) hide)
-    )
-    (pin "1")
-    (pin "2")
-  )
 )

Commit message: footprints added
Parts:
- IC2: footprint MLX90621ESFBAB000SP -> IRSensor:MLX90621ESFBAB000SP
Changed lines of the file:
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@@
     (property "Reference" "IC2" (id 0) (at 156.21 110.49 0))
     (property "Value" "MLX90621ESF-BAB-000-SP" (id 1) (at 156.21 113.03 0))
-    (property "Footprint" "MLX90621ESFBAB000SP" (id 2) (at 147.32 90.17 0)
+    (property "Footprint" "IRSensor:MLX90621ESFBAB000SP" (id 2) (at 147.32 90.17 0)
       (effects (font (size 1.27 1.27)) (justify left) hide)
     )
