File: hardware/TireTempSensor_v2.0/LEDs.kicad_sch (KiCad schematic)
At the start: 0 parts

Commit message: PFET & buck caps models
Parts:
- added D? (x2): RED, Diode_SMD:D_0603_1608Metric, symbol Device:D_Small
- added D? (x2): YELLOW, Diode_SMD:D_0603_1608Metric, symbol Device:D_Small
- added D?: GREEN, Diode_SMD:D_0603_1608Metric, symbol Device:D_Small
- added R? (x5): 1k5, Resistor_SMD:R_0603_1608Metric, symbol SB-Spoko-Bezpieczniki-rescue:R_Small-Device
Connections:
- new net: D?.1 (K), R?.1 (x5)
- new net +3V3: D?.2 (A)
- new net GND: R?.2, R?.2, R?.2, R?.2, R?.2
- new net LED_ERR: D?.2 (A)
- new net LED_OK: D?.2 (A)
- new net LED_WAR1: D?.2 (A)
- new net LED_WAR2: D?.2 (A)
Other:
- title: (none) -> LEDs

Commit message: erc tests passed
Parts:
- removed D? (x2): RED, Diode_SMD:D_0603_1608Metric, symbol Device:D_Small
- removed D? (x2): YELLOW, Diode_SMD:D_0603_1608Metric, symbol Device:D_Small
- removed D?: GREEN, Diode_SMD:D_0603_1608Metric, symbol Device:D_Small
- removed R? (x5): 1k5, Resistor_SMD:R_0603_1608Metric, symbol SB-Spoko-Bezpieczniki-rescue:R_Small-Device
- added D2, D6: RED, Diode_SMD:D_0603_1608Metric, symbol Device:D_Small
- added D3, D4: YELLOW, Diode_SMD:D_0603_1608Metric, symbol Device:D_Small
- added D5: GREEN, Diode_SMD:D_0603_1608Metric, symbol Device:D_Small
- added R10, R4, R7, R8, R9: 1k5, symbol Device:R_Small_US
Connections:
- net +3V3: now also R10.1
- net GND: now also D2.1 (K), D3.1 (K), D4.1 (K), D5.1 (K), D6.1 (K)
- net LED_ERR: now also R4.1
- net LED_OK: now also R9.1
- net LED_WAR1: now also R7.1
- net LED_WAR2: now also R8.1
- new net: D3.2 (A), R7.2
- new net: D4.2 (A), R8.2
- new net: D2.2 (A), R4.2
- new net: D6.2 (A), R10.2
- new net: D5.2 (A), R9.2

Commit message: footprints added
Parts:
- R10, R4, R7, R8, R9: footprint (none) -> Resistor_SMD:R_0603_1608Metric
Changed lines of the file:
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@@
       (effects (font (size 1.27 1.27)) (justify left))
     )
-    (property "Footprint" "" (id 2) (at 130.81 99.06 0)
+    (property "Footprint" "Resistor_SMD:R_0603_1608Metric" (id 2) (at 130.81 99.06 0)
       (effects (font (size 1.27 1.27)) hide)
     )
@@
       (effects (font (size 1.27 1.27)) (justify left))
     )
-    (property "Footprint" "" (id 2) (at 161.29 99.06 0)
+    (property "Footprint" "Resistor_SMD:R_0603_1608Metric" (id 2) (at 161.29 99.06 0)
       (effects (font (size 1.27 1.27)) hide)
     )
@@
       (effects (font (size 1.27 1.27)) (justify left))
     )
-    (property "Footprint" "" (id 2) (at 146.05 99.06 0)
+    (property "Footprint" "Resistor_SMD:R_0603_1608Metric" (id 2) (at 146.05 99.06 0)
       (effects (font (size 1.27 1.27)) hide)
     )
@@
       (effects (font (size 1.27 1.27)) (justify left))
     )
-    (property "Footprint" "" (id 2) (at 115.57 99.06 0)
+    (property "Footprint" "Resistor_SMD:R_0603_1608Metric" (id 2) (at 115.57 99.06 0)
       (effects (font (size 1.27 1.27)) hide)
     )
@@
       (effects (font (size 1.27 1.27)) (justify left))
     )
-    (property "Footprint" "" (id 2) (at 176.53 99.06 0)
-      (effects (font (size 1.27 1.27)) hide)
-    )
+    (property "Footprint" "Resistor_SMD:R_0603_1608Metric" (id 2) (at 176.53 99.06 0)
+      (effects (font (size 1.27 1.27)) hide)
+    )
