File: hardware/TireTempSensor_v2.0/CAN.kicad_sch (KiCad schematic)
At the start: 0 parts

Commit message: PFET & buck caps models
Parts:
- added D?: PESD2CAN,215, TSOT23-5:SOT-23, symbol Power_Protection:NUP2105L
- added FB?: 60R@100MHz, Inductor_SMD:L_0603_1608Metric, symbol Device:FerriteBead_Small
- added U?: SN65HVD232, Package_SO:SOIC-8_3.9x4.9mm_P1.27mm, symbol Interface_CAN_LIN:SN65HVD232
Connections:
- new net: FB?.2, U?.3 (VCC)
- new net +3V3: FB?.1
- new net CAN_H: D?.2 (K), U?.7 (CANH)
- new net CAN_L: D?.1 (K), U?.6 (CANL)
- new net CAN_RX: U?.4 (R)
- new net CAN_TX: U?.1 (D)
- new net GND: D?.3 (A), U?.2 (GND)
Changed lines of the file:
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@@
 (kicad_sch (version 20211123) (generator eeschema)
   (paper "A4")
+  (junction (at 134.62 90.17) (diameter 0) (color 0 0 0 0)
+  )
+  (wire (pts (xy 144.78 101.6) (xy 147.32 101.6))
+    (stroke (width 0) (type default) (color 0 0 0 0))
+  )
+  (wire (pts (xy 167.64 99.06) (xy 167.64 101.6))
+    (stroke (width 0) (type default) (color 0 0 0 0))
+  )
+  (wire (pts (xy 118.11 101.6) (xy 124.46 101.6))
+    (stroke (width 0) (type default) (color 0 0 0 0))
+  )
+  (wire (pts (xy 134.62 111.76) (xy 134.62 113.03))
+    (stroke (width 0) (type default) (color 0 0 0 0))
+  )
+  (wire (pts (xy 170.18 111.76) (xy 170.18 113.03))
+    (stroke (width 0) (type default) (color 0 0 0 0))
+  )
+  (wire (pts (xy 118.11 99.06) (xy 124.46 99.06))
+    (stroke (width 0) (type default) (color 0 0 0 0))
+  )
+  (wire (pts (xy 134.62 88.9) (xy 134.62 90.17))
+    (stroke (width 0) (type default) (color 0 0 0 0))
+  )
+  (wire (pts (xy 134.62 81.28) (xy 134.62 83.82))
+    (stroke (width 0) (type default) (color 0 0 0 0))
+  )
+  (wire (pts (xy 172.72 99.06) (xy 172.72 101.6))
+    (stroke (width 0) (type default) (color 0 0 0 0))
+  )
+  (wire (pts (xy 134.62 90.17) (xy 134.62 93.98))
+    (stroke (width 0) (type default) (color 0 0 0 0))
+  )
+  (wire (pts (xy 144.78 104.14) (xy 147.32 104.14))
+    (stroke (width 0) (type default) (color 0 0 0 0))
+  )
+  (wire (pts (xy 166.37 85.09) (xy 172.72 85.09))
+    (stroke (width 0) (type default) (color 0 0 0 0))
+  )
+  (wire (pts (xy 166.37 87.63) (xy 172.72 87.63))
+    (stroke (width 0) (type default) (color 0 0 0 0))
+  )
+  (label "CAN+" (at 166.37 85.09 180)
+    (effects (font (size 1.27 1.27)) (justify right bottom))
+  )
+  (label "CAN+" (at 147.32 101.6 0)
+    (effects (font (size 1.27 1.27)) (justify left bottom))
+  )
+  (label "CAN-" (at 166.37 87.63 180)
+    (effects (font (size 1.27 1.27)) (justify right bottom))
+  )
+  (label "CAN+" (at 172.72 99.06 0)
+    (effects (font (size 1.27 1.27)) (justify left bottom))
+  )
+  (label "CAN-" (at 167.64 99.06 180)
+    (effects (font (size 1.27 1.27)) (justify right bottom))
+  )
+  (label "CAN-" (at 147.32 104.14 0)
+    (effects (font (size 1.27 1.27)) (justify left bottom))
+  )
+  (hierarchical_label "CAN_TX" (shape input) (at 118.11 99.06 180)
+    (effects (font (size 1.27 1.27)) (justify right))
+  )
+  (hierarchical_label "CAN_L" (shape bidirectional) (at 172.72 87.63 0)
+    (effects (font (size 1.27 1.27)) (justify left))
+  )
+  (hierarchical_label "CAN_RX" (shape output) (at 118.11 101.6 180)
+    (effects (font (size 1.27 1.27)) (justify right))
+  )
+  (hierarchical_label "CAN_H" (shape bidirectional) (at 172.72 85.09 0)
+    (effects (font (size 1.27 1.27)) (justify left))
+  )
+  (symbol (lib_id "Power_Protection:NUP2105L") (at 170.18 106.68 0) (unit 1)
+    (in_bom yes) (on_board yes) (fields_autoplaced)
+    (property "Reference" "D?" (id 0) (at 176.53 105.4099 0)
+      (effects (font (size 1.27 1.27)) (justify left))
+    )
+    (property "Value" "PESD2CAN,215" (id 1) (at 176.53 107.9499 0)
+      (effects (font (size 1.27 1.27)) (justify left))
+    )
+    (property "Footprint" "TSOT23-5:SOT-23" (id 2) (at 175.895 107.95 0)
+      (effects (font (size 1.27 1.27)) (justify left) hide)
+    )
+    (property "Datasheet" "" (id 3) (at 173.355 103.505 0)
+      (effects (font (size 1.27 1.27)) hide)
+    )
+    (pin "3")
+    (pin "1")
+    (pin "2")
+  )
+  (symbol (lib_id "power:PWR_FLAG") (at 134.62 90.17 90) (unit 1)
+    (in_bom yes) (on_board yes) (fields_autoplaced)
+    (property "Reference" "#FLG?" (id 0) (at 132.715 90.17 0)
+      (effects (font (size 1.27 1.27)) hide)
+    )
+    (property "Value" "PWR_FLAG" (id 1) (at 129.54 90.17 0)
+      (effects (font (size 1.27 1.27)) hide)
+    )
+    (property "Footprint" "" (id 2) (at 134.62 90.17 0)
+      (effects (font (size 1.27 1.27)) hide)
+    )
+    (property "Datasheet" "~" (id 3) (at 134.62 90.17 0)
+      (effects (font (size 1.27 1.27)) hide)
+    )
+    (pin "1")
+  )
+  (symbol (lib_id "power:GND") (at 170.18 113.03 0) (unit 1)
+    (in_bom yes) (on_board yes) (fields_autoplaced)
+    (property "Reference" "#PWR?" (id 0) (at 170.18 119.38 0)
+      (effects (font (size 1.27 1.27)) hide)
+    )
+    (property "Value" "GND" (id 1) (at 170.18 118.11 0))
+    (property "Footprint" "" (id 2) (at 170.18 113.03 0)
+      (effects (font (size 1.27 1.27)) hide)
+    )
+    (property "Datasheet" "" (id 3) (at 170.18 113.03 0)
+      (effects (font (size 1.27 1.27)) hide)
+    )
+    (pin "1")
+  )
+  (symbol (lib_id "power:+3V3") (at 134.62 81.28 0) (unit 1)
+    (in_bom yes) (on_board yes) (fields_autoplaced)
+    (property "Reference" "#PWR?" (id 0) (at 134.62 85.09 0)
+      (effects (font (size 1.27 1.27)) hide)
+    )
+    (property "Value" "+3V3" (id 1) (at 134.62 76.2 0))
+    (property "Footprint" "" (id 2) (at 134.62 81.28 0)
+      (effects (font (size 1.27 1.27)) hide)
+    )
+    (property "Datasheet" "" (id 3) (at 134.62 81.28 0)
+      (effects (font (size 1.27 1.27)) hide)
+    )
+    (pin "1")
+  )
+  (symbol (lib_id "power:GND") (at 134.62 113.03 0) (unit 1)
+    (in_bom yes) (on_board yes) (fields_autoplaced)
+    (property "Reference" "#PWR?" (id 0) (at 134.62 119.38 0)
+      (effects (font (size 1.27 1.27)) hide)
+    )
+    (property "Value" "GND" (id 1) (at 134.62 118.11 0))
+    (property "Footprint" "" (id 2) (at 134.62 113.03 0)
+      (effects (font (size 1.27 1.27)) hide)
+    )
+    (property "Datasheet" "" (id 3) (at 134.62 113.03 0)
+      (effects (font (size 1.27 1.27)) hide)
+    )
+    (pin "1")
+  )
+  (symbol (lib_id "Device:FerriteBead_Small") (at 134.62 86.36 0) (unit 1)
+    (in_bom yes) (on_board yes)
+    (property "Reference" "FB?" (id 0) (at 127 85.09 0)
+      (effects (font (size 1.27 1.27)) (justify left))
+    )
+    (property "Value" "60R@100MHz" (id 1) (at 118.11 87.63 0)
+      (effects (font (size 1.27 1.27)) (justify left))
+    )
+    (property "Footprint" "Inductor_SMD:L_0603_1608Metric" (id 2) (at 132.842 86.36 90)
+      (effects (font (size 1.27 1.27)) hide)
+    )
+    (property "Datasheet" "~" (id 3) (at 134.62 86.36 0)
+      (effects (font (size 1.27 1.27)) hide)
+    )
+    (pin "1")
+    (pin "2")
+  )
+  (symbol (lib_id "Interface_CAN_LIN:SN65HVD232") (at 134.62 101.6 0) (unit 1)
+    (in_bom yes) (on_board yes)
+    (property "Reference" "U?" (id 0) (at 137.16 91.44 0)
+      (effects (font (size 1.27 1.27)) (justify left))
+    )
+    (property "Value" "SN65HVD232" (id 1) (at 136.6394 93.98 0)
+      (effects (font (size 1.27 1.27)) (justify left))
+    )
+    (property "Footprint" "Package_SO:SOIC-8_3.9x4.9mm_P1.27mm" (id 2) (at 134.62 114.3 0)
+      (effects (font (size 1.27 1.27)) hide)
+    )
+    (property "Datasheet" "http://www.ti.com/lit/ds/symlink/sn65hvd230.pdf" (id 3) (at 132.08 91.44 0)
+      (effects (font (size 1.27 1.27)) hide)
+    )
+    (pin "1")
+    (pin "2")
+    (pin "3")
+    (pin "4")
+    (pin "5")
+    (pin "6")
+    (pin "7")
+    (pin "8")
+  )
 )

Commit message: erc tests passed
Parts:
- gave numbers to parts that had none: 3
Other:
- moved on the sheet: D1
Changed lines of the file:
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@@
 (kicad_sch (version 20211123) (generator eeschema)
   (paper "A4")
+  (junction (at 152.4 101.6) (diameter 0) (color 0 0 0 0)
+  )
   (junction (at 134.62 90.17) (diameter 0) (color 0 0 0 0)
   )
-  (wire (pts (xy 144.78 101.6) (xy 147.32 101.6))
+  (junction (at 147.32 104.14) (diameter 0) (color 0 0 0 0)
+  )
+  (wire (pts (xy 152.4 101.6) (xy 152.4 105.41))
     (stroke (width 0) (type default) (color 0 0 0 0))
   )
-  (wire (pts (xy 167.64 99.06) (xy 167.64 101.6))
+  (wire (pts (xy 144.78 104.14) (xy 147.32 104.14))
     (stroke (width 0) (type default) (color 0 0 0 0))
   )
@@
     (stroke (width 0) (type default) (color 0 0 0 0))
   )
-  (wire (pts (xy 170.18 111.76) (xy 170.18 113.03))
+  (wire (pts (xy 149.86 115.57) (xy 149.86 116.84))
     (stroke (width 0) (type default) (color 0 0 0 0))
   )
@@
     (stroke (width 0) (type default) (color 0 0 0 0))
   )
-  (wire (pts (xy 134.62 81.28) (xy 134.62 83.82))
+  (wire (pts (xy 147.32 104.14) (xy 147.32 105.41))
     (stroke (width 0) (type default) (color 0 0 0 0))
   )
-  (wire (pts (xy 172.72 99.06) (xy 172.72 101.6))
+  (wire (pts (xy 134.62 81.28) (xy 134.62 83.82))
     (stroke (width 0) (type default) (color 0 0 0 0))
   )
@@
     (stroke (width 0) (type default) (color 0 0 0 0))
   )
-  (wire (pts (xy 144.78 104.14) (xy 147.32 104.14))
+  (wire (pts (xy 144.78 101.6) (xy 152.4 101.6))
     (stroke (width 0) (type default) (color 0 0 0 0))
   )
-  (wire (pts (xy 166.37 85.09) (xy 172.72 85.09))
+  (wire (pts (xy 152.4 101.6) (xy 158.75 101.6))
     (stroke (width 0) (type default) (color 0 0 0 0))
   )
-  (wire (pts (xy 166.37 87.63) (xy 172.72 87.63))
+  (wire (pts (xy 147.32 104.14) (xy 158.75 104.14))
     (stroke (width 0) (type default) (color 0 0 0 0))
-  )
-  (label "CAN+" (at 166.37 85.09 180)
-    (effects (font (size 1.27 1.27)) (justify right bottom))
-  )
-  (label "CAN+" (at 147.32 101.6 0)
-    (effects (font (size 1.27 1.27)) (justify left bottom))
-  )
-  (label "CAN-" (at 166.37 87.63 180)
-    (effects (font (size 1.27 1.27)) (justify right bottom))
-  )
-  (label "CAN+" (at 172.72 99.06 0)
-    (effects (font (size 1.27 1.27)) (justify left bottom))
-  )
-  (label "CAN-" (at 167.64 99.06 180)
-    (effects (font (size 1.27 1.27)) (justify right bottom))
-  )
-  (label "CAN-" (at 147.32 104.14 0)
-    (effects (font (size 1.27 1.27)) (justify left bottom))
   )
   (hierarchical_label "CAN_TX" (shape input) (at 118.11 99.06 180)
     (effects (font (size 1.27 1.27)) (justify right))
   )
-  (hierarchical_label "CAN_L" (shape bidirectional) (at 172.72 87.63 0)
+  (hierarchical_label "CAN_L" (shape bidirectional) (at 158.75 104.14 0)
     (effects (font (size 1.27 1.27)) (justify left))
   )
@@
     (effects (font (size 1.27 1.27)) (justify right))
   )
-  (hierarchical_label "CAN_H" (shape bidirectional) (at 172.72 85.09 0)
+  (hierarchical_label "CAN_H" (shape bidirectional) (at 158.75 101.6 0)
     (effects (font (size 1.27 1.27)) (justify left))
   )
-  (symbol (lib_id "Power_Protection:NUP2105L") (at 170.18 106.68 0) (unit 1)
+  (symbol (lib_id "Power_Protection:NUP2105L") (at 149.86 110.49 0) (unit 1)
     (in_bom yes) (on_board yes) (fields_autoplaced)
-    (property "Reference" "D?" (id 0) (at 176.53 105.4099 0)
+    (property "Reference" "D1" (id 0) (at 156.21 109.2199 0)
       (effects (font (size 1.27 1.27)) (justify left))
     )
-    (property "Value" "PESD2CAN,215" (id 1) (at 176.53 107.9499 0)
+    (property "Value" "PESD2CAN,215" (id 1) (at 156.21 111.7599 0)
       (effects (font (size 1.27 1.27)) (justify left))
     )
-    (property "Footprint" "TSOT23-5:SOT-23" (id 2) (at 175.895 107.95 0)
+    (property "Footprint" "TSOT23-5:SOT-23" (id 2) (at 155.575 111.76 0)
       (effects (font (size 1.27 1.27)) (justify left) hide)
     )
-    (property "Datasheet" "" (id 3) (at 173.355 103.505 0)
+    (property "Datasheet" "" (id 3) (at 153.035 107.315 0)
       (effects (font (size 1.27 1.27)) hide)
     )
@@
   (symbol (lib_id "power:PWR_FLAG") (at 134.62 90.17 90) (unit 1)
     (in_bom yes) (on_board yes) (fields_autoplaced)
-    (property "Reference" "#FLG?" (id 0) (at 132.715 90.17 0)
+    (property "Reference" "#FLG0105" (id 0) (at 132.715 90.17 0)
       (effects (font (size 1.27 1.27)) hide)
     )
@@
     (pin "1")
   )
-  (symbol (lib_id "power:GND") (at 170.18 113.03 0) (unit 1)
+  (symbol (lib_id "power:GND") (at 149.86 116.84 0) (unit 1)
     (in_bom yes) (on_board yes) (fields_autoplaced)
-    (property "Reference" "#PWR?" (id 0) (at 170.18 119.38 0)
+    (property "Reference" "#PWR0130" (id 0) (at 149.86 123.19 0)
       (effects (font (size 1.27 1.27)) hide)
     )
-    (property "Value" "GND" (id 1) (at 170.18 118.11 0))
-    (property "Footprint" "" (id 2) (at 170.18 113.03 0)
+    (property "Value" "GND" (id 1) (at 149.86 121.92 0))
+    (property "Footprint" "" (id 2) (at 149.86 116.84 0)
       (effects (font (size 1.27 1.27)) hide)
     )
-    (property "Datasheet" "" (id 3) (at 170.18 113.03 0)
+    (property "Datasheet" "" (id 3) (at 149.86 116.84 0)
       (effects (font (size 1.27 1.27)) hide)
     )
@@
   (symbol (lib_id "power:+3V3") (at 134.62 81.28 0) (unit 1)
     (in_bom yes) (on_board yes) (fields_autoplaced)
-    (property "Reference" "#PWR?" (id 0) (at 134.62 85.09 0)
+    (property "Reference" "#PWR0131" (id 0) (at 134.62 85.09 0)
       (effects (font (size 1.27 1.27)) hide)
     )
@@
   (symbol (lib_id "power:GND") (at 134.62 113.03 0) (unit 1)
     (in_bom yes) (on_board yes) (fields_autoplaced)
-    (property "Reference" "#PWR?" (id 0) (at 134.62 119.38 0)
+    (property "Reference" "#PWR0129" (id 0) (at 134.62 119.38 0)
       (effects (font (size 1.27 1.27)) hide)
     )
@@
   (symbol (lib_id "Device:FerriteBead_Small") (at 134.62 86.36 0) (unit 1)
     (in_bom yes) (on_board yes)
-    (property "Reference" "FB?" (id 0) (at 127 85.09 0)
+    (property "Reference" "FB4" (id 0) (at 127 85.09 0)
       (effects (font (size 1.27 1.27)) (justify left))
     )
@@
   (symbol (lib_id "Interface_CAN_LIN:SN65HVD232") (at 134.62 101.6 0) (unit 1)
     (in_bom yes) (on_board yes)
-    (property "Reference" "U?" (id 0) (at 137.16 91.44 0)
+    (property "Reference" "U3" (id 0) (at 137.16 91.44 0)
       (effects (font (size 1.27 1.27)) (justify left))
     )

Commit message: rough pcb layout
Parts:
- D1: footprint TSOT23-5:SOT-23 -> Package_TO_SOT_SMD:SOT-23
Changed lines of the file:
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@@
       (effects (font (size 1.27 1.27)) (justify left))
     )
-    (property "Footprint" "TSOT23-5:SOT-23" (id 2) (at 155.575 111.76 0)
+    (property "Footprint" "Package_TO_SOT_SMD:SOT-23" (id 2) (at 155.575 111.76 0)
       (effects (font (size 1.27 1.27)) (justify left) hide)
     )
