File: hardware/TireTempSensor_v2.0/TireTempSensor_v2.0.kicad_pcb (KiCad board)
At the start: 4 copper layers, 27 x 54 mm, 57 parts, among them IC1 MAX15462AATA+, IC2 MLX90621ESF-BAB-000-SP, J1 SWD_01x06, J2 CAN_01x04, Q1 FQT3P20TF, SW1 RESET, U1 STM32L4P5RET6, U2 MIC5306-2.6YD5-TR, U3 SN65HVD232, Y1 16MGHz

Commit message: Restructure code
Parts:
- J1: moved to F.Cu
- turned J1 to 0 degrees
Changed lines of the file:
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@@
+    )
+  )
+  (footprint "Connector_PinHeader_2.54mm:PinHeader_1x06_P2.54mm_Vertical" (layer "F.Cu")
+    (at 123.5 82.75)
+    (descr "Through hole straight pin header, 1x06, 2.54mm pitch, single row")
+    (tags "Through hole pin header THT 1x06 2.54mm single row")
+    (property "Sheetfile" "File: TireTempSensor_v2.0.kicad_sch")
+    (property "Sheetname" "")
+    (attr through_hole)
+    (fp_text reference "J1" (at 0 -2.33) (layer "User.1")
+      (effects (font (size 1 1) (thickness 0.15)))
+    )
+    (fp_text value "SWD_01x06" (at 0 15.03) (layer "F.Fab")
+      (effects (font (size 1 1) (thickness 0.15)))
+    )
+    (fp_text user "${REFERENCE}" (at 0 6.35 90) (layer "F.Fab")
+      (effects (font (size 1 1) (thickness 0.15)))
+    )
+    (fp_line (start -1.8 -1.8) (end -1.8 14.5) (layer "F.CrtYd") (width 0.05))
+    (fp_line (start 1.8 14.5) (end 1.8 -1.8) (layer "F.CrtYd") (width 0.05))
+    (fp_line (start -1.8 14.5) (end 1.8 14.5) (layer "F.CrtYd") (width 0.05))
+    (fp_line (start 1.8 -1.8) (end -1.8 -1.8) (layer "F.CrtYd") (width 0.05))
+    (fp_line (start -1.27 -0.635) (end -0.635 -1.27) (layer "F.Fab") (width 0.1))
+    (fp_line (start 1.27 -1.27) (end 1.27 13.97) (layer "F.Fab") (width 0.1))
+    (fp_line (start -1.27 13.97) (end -1.27 -0.635) (layer "F.Fab") (width 0.1))
+    (fp_line (start -0.635 -1.27) (end 1.27 -1.27) (layer "F.Fab") (width 0.1))
+    (fp_line (start 1.27 13.97) (end -1.27 13.97) (layer "F.Fab") (width 0.1))
+    (pad "1" thru_hole rect (at 0 0) (size 1.7 1.7) (drill 1) (layers *.Cu *.Mask)
+      (net 10 "+3V3") (pinfunction "Pin_1") (pintype "passive"))
+    (pad "2" thru_hole oval (at 0 2.54) (size 1.7 1.7) (drill 1) (layers *.Cu *.Mask)
+      (net 25 "/SWCLK") (pinfunction "Pin_2") (pintype "passive"))
+    (pad "3" thru_hole oval (at 0 5.08) (size 1.7 1.7) (drill 1) (layers *.Cu *.Mask)
+      (net 2 "GND") (pinfunction "Pin_3") (pintype "passive"))
+    (pad "4" thru_hole oval (at 0 7.62) (size 1.7 1.7) (drill 1) (layers *.Cu *.Mask)
+      (net 26 "/SWDIO") (pinfunction "Pin_4") (pintype "passive"))
+    (pad "5" thru_hole oval (at 0 10.16) (size 1.7 1.7) (drill 1) (layers *.Cu *.Mask)
+      (net 5 "/NRST") (pinfunction "Pin_5") (pintype "passive"))
+    (pad "6" thru_hole oval (at 0 12.7) (size 1.7 1.7) (drill 1) (layers *.Cu *.Mask)
+      (net 27 "/SWO") (pinfunction "Pin_6") (pintype "passive"))
+    (model "${KICAD6_3DMODEL_DIR}/Connector_PinHeader_2.54mm.3dshapes/PinHeader_1x06_P2.54mm_Vertical.wrl"
+      (offset (xyz 0 0 0))
+      (scale (xyz 1 1 1))
+      (rotate (xyz 0 0 0))
     )
   )
@@
       (offset (xyz 0 0 0))
       (scale (xyz 1 1 1))
-      (rotate (xyz 0 0 0))
-    )
-  )
-  (footprint "Connector_PinHeader_2.54mm:PinHeader_1x06_P2.54mm_Vertical" (layer "B.Cu")
-    (at 123.5 82.75 180)
-    (descr "Through hole straight pin header, 1x06, 2.54mm pitch, single row")
-    (tags "Through hole pin header THT 1x06 2.54mm single row")
-    (property "Sheetfile" "File: TireTempSensor_v2.0.kicad_sch")
-    (property "Sheetname" "")
-    (attr through_hole)
-    (fp_text reference "J1" (at 0 2.33) (layer "User.1")
-      (effects (font (size 1 1) (thickness 0.15)))
-    )
-    (fp_text value "SWD_01x06" (at 0 -15.03) (layer "B.Fab")
-      (effects (font (size 1 1) (thickness 0.15)) (justify mirror))
-    )
-    (fp_text user "${REFERENCE}" (at 0 -6.35 90) (layer "B.Fab")
-      (effects (font (size 1 1) (thickness 0.15)) (justify mirror))
-    )
-    (fp_line (start -1.8 1.8) (end -1.8 -14.5) (layer "B.CrtYd") (width 0.05))
-    (fp_line (start 1.8 -14.5) (end 1.8 1.8) (layer "B.CrtYd") (width 0.05))
-    (fp_line (start -1.8 -14.5) (end 1.8 -14.5) (layer "B.CrtYd") (width 0.05))
-    (fp_line (start 1.8 1.8) (end -1.8 1.8) (layer "B.CrtYd") (width 0.05))
-    (fp_line (start -1.27 0.635) (end -0.635 1.27) (layer "B.Fab") (width 0.1))
-    (fp_line (start 1.27 1.27) (end 1.27 -13.97) (layer "B.Fab") (width 0.1))
-    (fp_line (start -1.27 -13.97) (end -1.27 0.635) (layer "B.Fab") (width 0.1))
-    (fp_line (start -0.635 1.27) (end 1.27 1.27) (layer "B.Fab") (width 0.1))
-    (fp_line (start 1.27 -13.97) (end -1.27 -13.97) (layer "B.Fab") (width 0.1))
-    (pad "1" thru_hole rect (at 0 0 180) (size 1.7 1.7) (drill 1) (layers *.Cu *.Mask)
-      (net 10 "+3V3") (pinfunction "Pin_1") (pintype "passive"))
-    (pad "2" thru_hole oval (at 0 -2.54 180) (size 1.7 1.7) (drill 1) (layers *.Cu *.Mask)
-      (net 25 "/SWCLK") (pinfunction "Pin_2") (pintype "passive"))
-    (pad "3" thru_hole oval (at 0 -5.08 180) (size 1.7 1.7) (drill 1) (layers *.Cu *.Mask)
-      (net 2 "GND") (pinfunction "Pin_3") (pintype "passive"))
-    (pad "4" thru_hole oval (at 0 -7.62 180) (size 1.7 1.7) (drill 1) (layers *.Cu *.Mask)
-      (net 26 "/SWDIO") (pinfunction "Pin_4") (pintype "passive"))
-    (pad "5" thru_hole oval (at 0 -10.16 180) (size 1.7 1.7) (drill 1) (layers *.Cu *.Mask)
-      (net 5 "/NRST") (pinfunction "Pin_5") (pintype "passive"))
-    (pad "6" thru_hole oval (at 0 -12.7 180) (size 1.7 1.7) (drill 1) (layers *.Cu *.Mask)
-      (net 27 "/SWO") (pinfunction "Pin_6") (pintype "passive"))
-    (model "${KICAD6_3DMODEL_DIR}/Connector_PinHeader_2.54mm.3dshapes/PinHeader_1x06_P2.54mm_Vertical.wrl"
-      (offset (xyz 0 0 0))
-      (scale (xyz 1 1 1))
